File: LPF.kicad_sch (KiCad schematic)
At the start: 7 parts, among them U1 LM358

Commit message: Add files via upload
Parts:
- U1: value LM358 -> LM358AP; footprint Package_SO:VSSOP-8_3x3mm_P0.65mm -> LM358AP:DIP794W45P254L959H508Q8; Part Number LM358DGKR -> LM358AP
Changed lines of the file:
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@@
 			)
 		)
-		(property "Value" "LM358"
+		(property "Value" "LM358AP"
 			(at 83.82 57.15 0)
 			(effects
@@
 			)
 		)
-		(property "Footprint" "Package_SO:VSSOP-8_3x3mm_P0.65mm"
+		(property "Footprint" "LM358AP:DIP794W45P254L959H508Q8"
 			(at 83.82 64.77 0)
 			(effects
@@
 			)
 		)
-		(property "Description" "General Purpose Amplifier 2 Circuit 8-VSSOP"
+		(property "Description" "General Purpose Amplifier 2 Circuit 8-PDIP"
 			(at 83.82 64.77 0)
 			(effects
@@
 			)
 		)
-		(property "Part Number" "LM358DGKR"
+		(property "Part Number" "LM358AP"
 			(at 83.82 64.77 0)
 			(effects
@@
 			)
 		)
-		(property "Value" "LM358"
-			(at 19.05 55.372 0)
+		(property "Value" "LM358AP"
+			(at 18.288 55.88 0)
 			(effects
 				(font
@@
 			)
 		)
-		(property "Footprint" "Package_SO:VSSOP-8_3x3mm_P0.65mm"
+		(property "Footprint" "LM358AP:DIP794W45P254L959H508Q8"
 			(at 20.32 54.61 0)
 			(effects
@@
 			)
 		)
-		(property "Description" "General Purpose Amplifier 2 Circuit 8-VSSOP"
+		(property "Description" "General Purpose Amplifier 2 Circuit 8-PDIP"
 			(at 20.32 54.61 0)
 			(effects
@@
 			)
 		)
-		(property "Part Number" "LM358DGKR"
+		(property "Part Number" "LM358AP"
 			(at 20.32 54.61 0)
 			(effects
@@
 			)
 		)
-		(property "Value" "LM358"
+		(property "Value" "LM358AP"
 			(at 80.01 25.146 0)
 			(effects
@@
 			)
 		)
-		(property "Footprint" "Package_SO:VSSOP-8_3x3mm_P0.65mm"
+		(property "Footprint" "LM358AP:DIP794W45P254L959H508Q8"
 			(at 80.01 31.75 0)
 			(effects
@@
 			)
 		)
-		(property "Description" "General Purpose Amplifier 2 Circuit 8-VSSOP"
+		(property "Description" "General Purpose Amplifier 2 Circuit 8-PDIP"
 			(at 80.01 31.75 0)
 			(effects
@@
 			)
 		)
-		(property "Part Number" "LM358DGKR"
+		(property "Part Number" "LM358AP"
 			(at 80.01 31.75 0)
 			(effects
