File: MyFirstBuck.kicad_pcb (KiCad board)
At the start: 2 copper layers, 130.8 x 135.6 mm, 46 parts, among them J1 Conn_01x01_Pin, J2 Conn_01x01_Pin, J3 Conn_01x01_Pin, J4 Conn_01x01_Pin, J5 Conn_01x01_Pin, Q1 IRF540NPBF, U1 LM358, U2 LAUNCHXL-F28379D, U3 UCC5304DWVR, U4 TMV 0512SHI

Commit message: Add files via upload
Parts:
- added REF**: MountingHole_2.2mm_M2, MountingHole:MountingHole_2.2mm_M2, F.Cu at (163.4, 180.3)
- added REF**: MountingHole_2.2mm_M2, MountingHole:MountingHole_2.2mm_M2, F.Cu at (163.4, 54.2)
- added REF**: MountingHole_2.2mm_M2, MountingHole:MountingHole_2.2mm_M2, F.Cu at (38.6, 54.2)
- added REF**: MountingHole_2.2mm_M2, MountingHole:MountingHole_2.2mm_M2, F.Cu at (38.5, 180.3)
- U1: value LM358 -> LM358AP; footprint Package_SO:VSSOP-8_3x3mm_P0.65mm -> LM358AP:DIP794W45P254L959H508Q8
- moved C2 12.5 mm to (140.1, 111.4)
- moved U1 11.7 mm to (143.1, 101.8)
- moved J5 11.5 mm to (86.2, 61.6)
- moved J1 11.4 mm to (43.0, 61.5)
- moved J3 11.4 mm to (159.0, 61.5)
- moved L3 10.6 mm to (136.0, 84.9)
- moved J2 8.92 mm to (43.0, 79.0)
- moved J4 8.92 mm to (159.0, 79.0)
- moved R4 8.12 mm to (152.5, 95.0)
- moved R7 6.29 mm to (148.3, 111.3), turned to 180 degrees
- moved C9 5.84 mm to (43.8, 90.5), turned to 90 degrees
- moved R13 5.59 mm to (56.5, 83.1)
- moved D4 5.18 mm to (147.9, 115.1), turned to 180 degrees
- moved C8 4.56 mm to (42.9, 95.0), turned to 180 degrees
- moved G*** 4.51 mm to (64.9, 66.2)
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Routing:
- net +5V: track 93.5 -> 66.1 mm
- net /VOUT: track 77.4 -> 61.1 mm
- net /VSW: track 155.3 -> 169.2 mm
- net Net-(U1A-+): track 7.68 -> 18.5 mm
- net /VFILT: track 53.4 -> 62.9 mm
- net Net-(U1A--): track 5.60 -> 14.8 mm
- net /VG: track 21.4 -> 29.4 mm
- net Net-(L2-Pad2): track 32.1 -> 38.0 mm
- net /GD/ISO_12: track 26.2 -> 31.1 mm
- net /PowerStage/VIN: track 78.9 -> 74.1 mm
- net /PWM: track 86.0 -> 89.4 mm
- net Net-(D7-K): track 2.28 -> 5.15 mm
- net /GD/GD_PWM: track 7.44 -> 8.96 mm
- net +3.3V: track 30.6 -> 29.2 mm
- net Net-(D4-K): track 2.65 -> 4.12 mm
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Other:
- board size 130.8 x 135.6 mm -> 130.8 x 132.1 mm
