File: MyFirstBuck.kicad_pcb (KiCad board)
At the start: 2 copper layers, 130.8 x 132.1 mm, 50 parts, among them J1 Conn_01x01_Pin, J2 Conn_01x01_Pin, J3 Conn_01x01_Pin, J4 Conn_01x01_Pin, J5 Conn_01x01_Pin, Q1 IRF540NPBF, U1 LM358AP, U2 LAUNCHXL-F28379D, U3 UCC5304DWVR, U4 TMV 0512SHI

Commit message: Add files via upload
Routing:
- net Net-(L1-Pad2): track 30.5 -> 29.5 mm
- net GND: vias 7 -> 6
Changed lines of the file:
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@@
 		)
 		(fp_text user "J7"
-			(at 28.075 20.412 0)
+			(at 28.075 20.082 0)
 			(layer "F.SilkS")
 			(effects
@@
 	)
 	(via
-		(at 39.1206 105.799)
+		(at 39.5 107.5)
 		(size 0.6)
 		(drill 0.3)
@@
 	)
 	(via
-		(at 38.257 102.751)
+		(at 38.5 102)
 		(size 0.6)
 		(drill 0.3)
@@
 	)
 	(via
-		(at 45.7246 101.227)
-		(size 0.6)
-		(drill 0.3)
-		(layers "F.Cu" "B.Cu")
-		(free yes)
-		(net 5)
-	)
-	(via
-		(at 43.6926 114.181)
+		(at 50.5 112)
 		(size 0.6)
 		(drill 0.3)
@@
 	)
 	(segment
-		(start 128.99 129.72)
-		(end 129.032 129.678)
+		(start 129.032 129.762)
+		(end 131.65 132.38)
 		(width 0.5)
 		(layer "F.Cu")
@@
 	)
 	(segment
-		(start 129.032 129.678)
-		(end 129.032 127.762)
-		(width 0.5)
-		(layer "F.Cu")
-		(net 8)
-	)
-	(segment
 		(start 131.65 132.38)
-		(end 128.99 129.72)
+		(end 152.28 132.38)
 		(width 0.5)
 		(layer "F.Cu")
@@
 	)
 	(segment
-		(start 152.28 132.38)
-		(end 131.65 132.38)
+		(start 156.62 128.04)
+		(end 156.62 108.37)
 		(width 0.5)
 		(layer "F.Cu")
@@
 	)
 	(segment
-		(start 156.62 128.04)
-		(end 152.28 132.38)
+		(start 129.032 127.762)
+		(end 129.032 129.762)
 		(width 0.5)
 		(layer "F.Cu")
@@
 	)
 	(segment
-		(start 156.62 108.37)
+		(start 152.28 132.38)
 		(end 156.62 128.04)
 		(width 0.5)
@@
 	)
 	(segment
-		(start 68.455 117.98)
-		(end 68.455 116.02)
-		(width 0.5)
-		(layer "F.Cu")
-		(net 15)
-	)
-	(segment
-		(start 68.454 117.979)
-		(end 68.455 117.98)
+		(start 73.238 127.762)
+		(end 73.5 127.5)
 		(width 0.5)
 		(layer "F.Cu")
@@
 	)
 	(segment
-		(start 52.1956 117.979)
-		(end 68.454 117.979)
-		(width 0.5)
-		(layer "F.Cu")
-		(net 15)
-	)
-	(segment
-		(start 72.81 123.0375)
-		(end 68.455 118.6825)
+		(start 70.612 127.762)
+		(end 73.238 127.762)
 		(width 0.5)
 		(layer "F.Cu")
@@
 	)
 	(segment
-		(start 52.1956 117.979)
+		(start 50.2366 116.02)
 		(end 44.4056 110.189)
 		(width 0.5)
@@
 	)
 	(segment
-		(start 70.612 127.762)
-		(end 72.762 127.762)
+		(start 73.5 127.5)
+		(end 73.5 121.065)
 		(width 0.5)
 		(layer "F.Cu")
@@
 	)
 	(segment
-		(start 72.81 127.81)
-		(end 72.81 123.0375)
-		(width 0.5)
-		(layer "F.Cu")
-		(net 15)
-	)
-	(segment
 		(start 47.405 95.695)
 		(end 48.5652 95.695)
@@
 	)
 	(segment
-		(start 72.762 127.762)
-		(end 72.81 127.81)
+		(start 68.455 116.02)
+		(end 50.2366 116.02)
 		(width 0.5)
 		(layer "F.Cu")
@@
 	)
 	(segment
-		(start 68.455 118.6825)
-		(end 68.455 117.98)
+		(start 73.5 121.065)
+		(end 68.455 116.02)
 		(width 0.5)
 		(layer "F.Cu")
@@
 	)
 	(segment
-		(start 59.6456 106.7631)
-		(end 59.3525 106.47)
-		(width 1)
-		(layer "F.Cu")
-		(net 17)
-	)
-	(segment
 		(start 56.0475 100.55)
 		(end 56.0475 94.5914)
@@
 	)
 	(segment
+		(start 59.6456 106.7631)
+		(end 59.3525 106.47)
+		(width 1)
+		(layer "F.Cu")
+		(net 17)
+	)
+	(segment
 		(start 59.6456 110.189)
 		(end 59.6456 106.7631)
@@
 	)
 	(segment
+		(start 61.4575 99.0877)
+		(end 59.3348 96.965)
+		(width 1)
+		(layer "F.Cu")
+		(net 33)
+	)
+	(segment
 		(start 59.3348 96.965)
 		(end 59.3348 95.695)
@@
 	)
 	(segment
-		(start 61.4575 100.54)
-		(end 61.4575 99.0877)
-		(width 1)
-		(layer "F.Cu")
-		(net 33)
-	)
-	(segment
 		(start 54.5656 110.189)
 		(end 57.3384 112.9618)
@@
 	)
 	(segment
-		(start 96.1644 92.369)
-		(end 105.6266 101.8312)
+		(start 96.369 92.369)
+		(end 105.6266 101.6266)
 		(width 1)
 		(layer "F.Cu")
@@
 	)
 	(segment
-		(start 61.4575 99.0877)
-		(end 59.3348 96.965)
-		(width 1)
+		(start 60.9138 112.9618)
+		(end 61.4275 112.4481)
+		(width 0.5)
 		(layer "F.Cu")
 		(net 33)
 	)
 	(segment
-		(start 60.9138 112.9618)
-		(end 61.4275 112.4481)
-		(width 0.5)
+		(start 96.1644 92.369)
+		(end 96.369 92.369)
+		(width 1)
 		(layer "F.Cu")
 		(net 33)
@@
 	)
 	(segment
-		(start 84.0232 88.7568)
-		(end 86.19 86.59)
-		(width 0.5)
+		(start 61.4575 100.54)
+		(end 61.4575 99.0877)
+		(width 1)
 		(layer "F.Cu")
 		(net 33)
 	)
 	(segment
-		(start 105.6266 101.8312)
+		(start 105.6266 101.6266)
 		(end 105.6266 104.0638)
 		(width 1)
@@
 	)
 	(segment
+		(start 84.0232 88.7568)
+		(end 86.19 86.59)
+		(width 0.5)
+		(layer "F.Cu")
+		(net 33)
+	)
+	(segment
 		(start 79.5062 92.6138)
 		(end 72.7 99.42)
@@
 	)
 	(segment
-		(start 37.1394 114.2394)
-		(end 45.09 122.19)
+		(start 37.1394 105.545)
+		(end 38.1127 105.545)
 		(width 0.5)
 		(layer "F.Cu")
@@
 	)
 	(segment
-		(start 38.7142 103.9702)
-		(end 37.1394 105.545)
+		(start 37.1394 114.2394)
+		(end 45.09 122.19)
 		(width 0.5)
 		(layer "F.Cu")
@@
 	)
 	(segment
-		(start 39.775 103.9702)
-		(end 38.7142 103.9702)
+		(start 38.1127 105.545)
+		(end 39.6875 103.9702)
 		(width 0.5)
 		(layer "F.Cu")
@@
 		(width 1)
 		(layer "F.Cu")
-		(net 112)
-	)
-	(segment
-		(start 106.7794 84.9762)
-		(end 105.7648 84.9762)
-		(width 1)
-		(layer "F.Cu")
