File: MyFirstBuck.kicad_pcb (KiCad board)
At the start: 2 copper layers, 130.8 x 132.1 mm, 50 parts, among them J1 Conn_01x01_Pin, J2 Conn_01x01_Pin, J3 Conn_01x01_Pin, J4 Conn_01x01_Pin, J5 Conn_01x01_Pin, Q1 IRF540NPBF, U1 LM358AP, U2 LAUNCHXL-F28379D, U3 UCC5304DWVR, U4 TMV 0512SHI

Commit message: Add files via upload
Other:
- board text added: "Fullmetal Buck Converter v0 - 01 Mar 2025 Manveer Aujla Alice Seo"
- board text removed: "Fullmetal Buck Converter v0 - 24 Feb 2025 Manveer Aujla Alice Seo"
Changed lines of the file:
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@@
 		)
 	)
-	(gr_text "Fullmetal Buck Converter\nv0 - 24 Feb 2025\nManveer Aujla\nAlice Seo"
+	(gr_text "Fullmetal Buck Converter\nv0 - 01 Mar 2025\nManveer Aujla\nAlice Seo"
 		(at 53 77.2 0)
 		(layer "F.SilkS")

Commit message: Add files via upload
Parts:
- L1, L2, L3: footprint Inductor_THT:L_Radial_D24.4mm_P23.90mm_Murata_1400series -> Inductor_THT:L_Radial_D24.4mm_P23.10mm_Murata_1400series
Routing:
- net Net-(L1-Pad2): track 29.5 -> 28.7 mm

Commit message: Add files via upload
Routing:
- net /VSW: track 169.4 -> 156.2 mm
Changed lines of the file:
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@@
-	)
-	(segment
-		(start 146.3179 115.09)
-		(end 146.504 115.09)
-		(width 0.2)
-		(layer "F.Cu")
-		(net 6)
 	)
 	(segment
@@
 	)
 	(segment
-		(start 84.0582 62.9418)
-		(end 86 61)
-		(width 0.2)
-		(layer "F.Cu")
-		(net 33)
-	)
-	(segment
 		(start 52.489 110.189)
 		(end 49.99 107.69)
@@
 	)
 	(segment
-		(start 84.0232 63.2968)
-		(end 86.16 61.16)
-		(width 0.5)
-		(layer "F.Cu")
-		(net 33)
-	)
-	(segment
-		(start 84.0232 62.9768)
-		(end 86 61)
-		(width 0.5)
-		(layer "F.Cu")
-		(net 33)
-	)
-	(segment
 		(start 61.4575 100.54)
 		(end 61.4575 99.0877)
@@
 		(end 55.54 83.71)
 		(width 0.5)
-		(layer "F.Cu")
-		(net 33)
-	)
-	(segment
-		(start 82.784 64.216)
-		(end 86 61)
-		(width 0.2)
 		(layer "F.Cu")
 		(net 33)
@@
 	)
 	(segment
-		(start 149.05 114.836)
-		(end 149.304 115.09)
-		(width 0.2)
-		(layer "F.Cu")
-		(net 60)
-	)
-	(segment

Commit message: Add files via upload
Parts:
- removed the REF** at (163.4, 180.3)
- removed the REF** at (163.4, 54.2)
- removed the REF** at (38.6, 54.2)
- removed the REF** at (38.5, 180.3)
- added REF**: MountingHole_2.7mm_M2.5, MountingHole:MountingHole_2.7mm_M2.5, F.Cu at (162.8, 180.8)
- added REF**: MountingHole_2.7mm_M2.5, MountingHole:MountingHole_2.7mm_M2.5, F.Cu at (39.0, 180.8)
- added REF**: MountingHole_2.7mm_M2.5, MountingHole:MountingHole_2.7mm_M2.5, F.Cu at (162.8, 53.4)
- added REF**: MountingHole_2.7mm_M2.5, MountingHole:MountingHole_2.7mm_M2.5, F.Cu at (39.1, 53.4)
Other:
- board size 130.8 x 132.1 mm -> 130.8 x 134.4 mm
