File: PowerStage.kicad_sch (KiCad schematic)
At the start: 13 parts, among them J1 Conn_01x01_Pin, J2 Conn_01x01_Pin, J3 Conn_01x01_Pin, J4 Conn_01x01_Pin, J5 Conn_01x01_Pin, Q1 IRF540NPBF

Commit message: Add files via upload
Parts:
- L1, L2, L3: footprint Inductor_THT:L_Radial_D24.4mm_P23.90mm_Murata_1400series -> Inductor_THT:L_Radial_D24.4mm_P23.10mm_Murata_1400series
Changed lines of the file:
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@@
 			)
 		)
-		(property "Footprint" "Inductor_THT:L_Radial_D24.4mm_P23.90mm_Murata_1400series"
+		(property "Footprint" "Inductor_THT:L_Radial_D24.4mm_P23.10mm_Murata_1400series"
 			(at 107.95 30.48 0)
 			(effects
@@
 			)
 		)
-		(property "Footprint" "Inductor_THT:L_Radial_D24.4mm_P23.90mm_Murata_1400series"
+		(property "Footprint" "Inductor_THT:L_Radial_D24.4mm_P23.10mm_Murata_1400series"
 			(at 97.79 30.48 0)
 			(effects
@@
 			)
 		)
-		(property "Footprint" "Inductor_THT:L_Radial_D24.4mm_P23.90mm_Murata_1400series"
+		(property "Footprint" "Inductor_THT:L_Radial_D24.4mm_P23.10mm_Murata_1400series"
 			(at 118.11 30.48 0)
 			(effects
